File: Quadraphone_Controls.kicad_sch (KiCad schematic)
At the start: 32 parts, among them J1 Eurorack_10_pin_power, SW1 SYNCH_SWITCH, SW2 DPDT_Switch, U1 AMS1117-5.0, U10 TL074, U14 TL074, U19 TL074, U2 MCP1501-25xSN, U4 LM4040DBZ-5, U5 MCP6004, U8 4066

Commit message: Started PCB layout
Parts:
- removed C1: 1nF, Capacitor_SMD:C_0603_1608Metric_Pad1.08x0.95mm_HandSolder, symbol Device:C_Small
- removed C10: 100nF, Capacitor_SMD:C_0603_1608Metric_Pad1.08x0.95mm_HandSolder, symbol Device:C_Small
- removed C11: 47uF, Capacitor_SMD:CP_Elec_5x5.8, symbol Device:C_Polarized_Small
- removed C12: 22uF, Capacitor_SMD:CP_Elec_4x5.8, symbol Device:C_Polarized_Small
- removed C2, C3: 10uF, Capacitor_SMD:CP_Elec_5x5.7, symbol Device:C_Polarized_Small
- removed C9: 1uF, Capacitor_SMD:C_0805_2012Metric, symbol Device:C_Small
- removed D1, D2: 1N5819, Diode_SMD:D_SOD-123, symbol Diode:1N5819
- removed J1: Eurorack_10_pin_power, Custom_Footprints:Eurorack_10_pin_header, symbol Eurorack_Header:Eurorack_10_pin_power
- removed R1, R10, R2, R3, R6: 14k, Resistor_SMD:R_0603_1608Metric, symbol Device:R_Small
- removed R13: 2.2k, Resistor_SMD:R_0603_1608Metric, symbol Device:R_Small
- removed U1: AMS1117-5.0, Package_TO_SOT_SMD:SOT-223-3_TabPin2, symbol Regulator_Linear:AMS1117-5.0
- removed U10, U14, U19: TL074, Package_SO:SOIC-14_3.9x8.7mm_P1.27mm, symbol Amplifier_Operational:TL074
- removed U2: MCP1501-25xSN, Package_SO:SOIC-8_3.9x4.9mm_P1.27mm, symbol Reference_Voltage:MCP1501-25xSN
- removed U4: LM4040DBZ-5, Package_TO_SOT_SMD:SOT-23, symbol Reference_Voltage:LM4040DBZ-5
- removed U5: MCP6004, Package_SO:SOIC-14_3.9x8.7mm_P1.27mm, symbol Amplifier_Operational:MCP6004
- removed U8: 4066, Package_SO:TSSOP-14_4.4x5mm_P0.65mm, symbol 4xxx:4066
Other:
- removed sheet OSCVoice1
- removed sheet OSCVoice2
- removed sheet OSCVoice3
- removed sheet OSCVoice4
- moved on the sheet: PWM_Pot1, SW1, SW2, Vibrato_Depth1
