File: _autosave-Quadraphone.kicad_pcb (KiCad board)
At the start: 2 copper layers, 60 x 110 mm, 164 parts, among them J1 Conn_01x10_Male, J2 Conn_01x10_Male, J3 Conn_01x10_Male, J4 Conn_01x10_Male, J5 Eurorack_10_pin_power, U1 AMS1117-5.0, U10 TL074, U11 4066, U12 SSI2131, U14 TL074, U15 4066, U17 SSI2131, U19 TL074, U2 MCP1501-25xSN, U22 SSI2131, U4 LM4040DBZ-5, U5 MCP6004, U6 4066, U7 4066, U8 4066, U9 SSI2131

Commit message: Started PCB layout
Parts:
- renumbered R7 to Expo_Trim1, R37 to Expo_Trim2, R83 to Expo_Trim3, R60 to Expo_Trim4, HF_Track_Trim4 to HF_Track_Trim3, HF_Track_Trim3 to HF_Track_Trim4
Connections:
- net /OSCVoice1/PULSE_MIX renamed /OSCVoice1/Pulse_Mix
- net /OSCVoice1/SAW_MIX renamed /OSCVoice1/Saw_Mix
- net /OSCVoice1/TRI_MIX renamed /OSCVoice1/Triangle_Mix
- net /OSCVoice2/PULSE_MIX renamed /OSCVoice2/Pulse_Mix
- net /OSCVoice2/SAW_MIX renamed /OSCVoice2/Saw_Mix
- net /OSCVoice2/TRI_MIX renamed /OSCVoice2/Triangle_Mix
- net /OSCVoice3/PULSE_MIX renamed /OSCVoice3/Pulse_Mix
- net /OSCVoice3/SAW_MIX renamed /OSCVoice3/Saw_Mix
- net /OSCVoice3/TRI_MIX renamed /OSCVoice3/Triangle_Mix
- net /OSCVoice4/PULSE_MIX renamed /OSCVoice4/Pulse_Mix
- net /OSCVoice4/SAW_MIX renamed /OSCVoice4/Saw_Mix
- net /OSCVoice4/TRI_MIX renamed /OSCVoice4/Triangle_Mix
