File: Quadraphone_Panel.kicad_pcb (KiCad board)
At the start: 2 copper layers, 60.8 x 128.5 mm, 17 parts, among them J10 Pitch_In, J11 Mix_Out, J7 PWM_CV_In, J8 Synch_Signal_In, J9 Freq_Mod_In

Commit message: Rough Layout of Panel
Parts:
- removed J10: Pitch_In, Custom_Footprints:RJ45_Molex_42878-8506
- removed J11: Mix_Out, Custom_Footprints:RJ45_Molex_42878-8506
- removed J7: PWM_CV_In, Custom_Footprints:RJ45_Molex_42878-8506
- removed J8: Synch_Signal_In, Custom_Footprints:RJ45_Molex_42878-8506
- removed J9: Freq_Mod_In, Custom_Footprints:RJ45_Molex_42878-8506
- added FM_In: RJ45_Molex_42878-8506_Mounting_Hole, Custom_Footprints:RJ45_Molex_42878-8506_Mounting_Hole, F.Cu at (62.2, 124.9)
- added Output: RJ45_Molex_42878-8506_Mounting_Hole, Custom_Footprints:RJ45_Molex_42878-8506_Mounting_Hole, F.Cu at (91.1, 143.9)
- added PWM_In: RJ45_Molex_42878-8506_Mounting_Hole, Custom_Footprints:RJ45_Molex_42878-8506_Mounting_Hole, F.Cu at (80.0, 124.9)
- added Synch_In: RJ45_Molex_42878-8506_Mounting_Hole, Custom_Footprints:RJ45_Molex_42878-8506_Mounting_Hole, F.Cu at (97.8, 124.9)
- added V_per_Oct_In: RJ45_Molex_42878-8506_Mounting_Hole, Custom_Footprints:RJ45_Molex_42878-8506_Mounting_Hole, F.Cu at (68.9, 143.9)
Other:
- board text added: "FM In"
- board text added: "Output"
- board text added: "PWM In"
- board text added: "Synch In"
- board text added: "V/Oct"

Commit message: First draft panel done
Parts:
- added G***: LOGO, Graphics:QuadraphoneLogo, F.Cu at (80.0, 39.9)
- added kibuzzard-63D0FD70: G***, kibuzzard-63D0FD70, F.Cu at (102.0, 76.0)
- added kibuzzard-63D12295: G***, kibuzzard-63D12295, F.Cu at (66.0, 47.0)
- added kibuzzard-63D122C1: G***, kibuzzard-63D122C1, F.Cu at (94.0, 47.0)
- added kibuzzard-63D122DE: G***, kibuzzard-63D122DE, F.Cu at (58.0, 76.0)
- added kibuzzard-63D127EA: G***, kibuzzard-63D127EA, F.Cu at (80.0, 57.0)
- added kibuzzard-63D12809: G***, kibuzzard-63D12809, F.Cu at (96.0, 106.6)
- added kibuzzard-63D1286A: G***, kibuzzard-63D1286A, F.Cu at (88.9, 69.9)
- added kibuzzard-63D1288B: G***, kibuzzard-63D1288B, F.Cu at (88.9, 82.1)
- added kibuzzard-63D139E5: G***, kibuzzard-63D139E5, F.Cu at (58.0, 109.0)
- added kibuzzard-63D139F5: G***, kibuzzard-63D139F5, F.Cu at (62.0, 134.5)
- added kibuzzard-63D13A10: G***, kibuzzard-63D13A10, F.Cu at (98.5, 134.5)
- added kibuzzard-63D1404C: G***, kibuzzard-63D1404C, F.Cu at (80.0, 100.1)
- moved Ref** 31.1 mm to (80.0, 125.0)
- moved Ref** 22.6 mm to (80.0, 109.0)
- moved Ref** 21.6 mm to (64.0, 94.0)
- moved Synch_In 21.1 mm to (98.4, 146.0)
- moved Ref** 17.9 mm to (96.0, 94.0)
- moved PWM_In 16.5 mm to (96.0, 121.0)
- moved Output 11.3 mm to (80.0, 146.0)
- moved V_per_Oct_In 7.60 mm to (61.6, 146.0)
- moved Ref** 4.33 mm to (94.0, 76.0)
- moved Ref** 4.30 mm to (66.0, 76.0)
- moved FM_In 4.30 mm to (64.0, 121.0)
- moved Ref** 0.59 mm to (94.0, 57.0)
- moved Ref** 0.54 mm to (66.0, 57.0)
Other:
- board text removed: "Coarse Tune"
- board text removed: "FM In"
- board text removed: "Fine Tune"
- board text removed: "Hard Synch"
- board text removed: "Output"
- board text removed: "PWM"
- board text removed: "PWM In"
- board text removed: "Soft Synch"
- board text removed: "Synch In"
- board text removed: "V/Oct"
- board text removed: "Vibrato"
- board text removed: "Vibrato Depth"
