File: Quadraphone_Breakout_Controls.kicad_sch (KiCad schematic)
At the start: 10 parts, among them J1 Mult_A, J10 JackB4, J2 Mult_B, J3 JackA1, J4 JackA2, J5 JackA3, J6 JackA4, J7 JackB1, J8 JackB2, J9 JackB3

Commit message: Prepared all gerbers
Parts:
- added J11, J12: Conn_02x04_Top_Bottom, Connector_PinHeader_2.54mm:PinHeader_2x04_P2.54mm_Vertical, symbol Connector_Generic:Conn_02x04_Odd_Even
Connections:
- net A1: now also J11.1 (Pin_1)
- net A2: now also J11.3 (Pin_3)
- net A3: now also J11.5 (Pin_5)
- net A4: now also J11.7 (Pin_7)
- net B1: now also J12.1 (Pin_1)
- net B2: now also J12.3 (Pin_3)
- net B3: now also J12.5 (Pin_5)
- net B4: now also J12.7 (Pin_7)
- net B5: now reaches J2.5
- net B5: now also J12.2 (Pin_2)
- net B6: now reaches J2.6
- net B6: now also J12.4 (Pin_4)
- net B7: now reaches J2.7
- net B7: now also J12.6 (Pin_6)
- net B8: now reaches J2.8
- net B8: now also J12.8 (Pin_8)
- net A5: now reaches J1.5
- net A5: now also J11.2 (Pin_2)
- net A6: now reaches J1.6
- net A6: now also J11.4 (Pin_4)
- net A7: now reaches J1.7
- net A7: now also J11.6 (Pin_6)
- net A8: now reaches J1.8
- net A8: now also J11.8 (Pin_8)
- no-connect marks 16 -> 8
