File: Quadraphone_Breakout_Panel.kicad_pcb (KiCad board)
At the start: 2 copper layers, 20.3 x 128.5 mm, 22 parts

Commit message: Prepared all gerbers
Parts:
- removed kibuzzard-63D415A8: G***, kibuzzard-63D415A8
- removed kibuzzard-63D415BB: G***, kibuzzard-63D415BB
- removed kibuzzard-63D415F2 (x2): G***, kibuzzard-63D415F2
- removed kibuzzard-63D4160B (x2): G***, kibuzzard-63D4160B
- removed kibuzzard-63D41618 (x2): G***, kibuzzard-63D41618
- removed kibuzzard-63D41624 (x2): G***, kibuzzard-63D41624
- added kibuzzard-63D64BAD: G***, kibuzzard-63D64BAD, F.Cu at (59.4, 54.1)
- added kibuzzard-63D64BB9: G***, kibuzzard-63D64BB9, F.Cu at (54.8, 87.9)
- added kibuzzard-63D64BC1: G***, kibuzzard-63D64BC1, F.Cu at (64.0, 87.9)
- added kibuzzard-63D64BC6: G***, kibuzzard-63D64BC6, F.Cu at (54.8, 102.8)
- added kibuzzard-63D64BCB: G***, kibuzzard-63D64BCB, F.Cu at (64.0, 102.8)
- added kibuzzard-63D64BCE: G***, kibuzzard-63D64BCE, F.Cu at (59.4, 108.1)
- added kibuzzard-63D64BD4: G***, kibuzzard-63D64BD4, F.Cu at (54.8, 141.3)
- added kibuzzard-63D64BD7: G***, kibuzzard-63D64BD7, F.Cu at (64.0, 141.3)
- added kibuzzard-63D64BDC: G***, kibuzzard-63D64BDC, F.Cu at (54.8, 156.2)
- added kibuzzard-63D64BE0: G***, kibuzzard-63D64BE0, F.Cu at (64.0, 156.2)
- moved FM_In 2.05 mm to (59.4, 65.0)
- moved Ref** 2.00 mm to (64.0, 81.0)
- moved Ref** 2.00 mm to (54.8, 81.0)
- moved Ref** 2.00 mm to (54.8, 96.0)
- moved Ref** 2.00 mm to (64.0, 96.0)
Other:
- board text added: "Breakout"
- board text added: "Mountjoy"
- board text removed: "Mountjoy Modular"
