File: Quadraphone_Breakout_Controls.kicad_pcb (KiCad board)
At the start: 2 copper layers, 18.8 x 110 mm, 10 parts, among them J1 Mult_A, J10 JackB4, J2 Mult_B, J3 JackA1, J4 JackA2, J5 JackA3, J6 JackA4, J7 JackB1, J8 JackB2, J9 JackB3

Commit message: Prepared all gerbers
Parts:
- added J11: Conn_02x04_Top_Bottom, Connector_PinHeader_2.54mm:PinHeader_2x04_P2.54mm_Vertical, B.Cu at (55.6, 51.9)
- added J12: Conn_02x04_Top_Bottom, Connector_PinHeader_2.54mm:PinHeader_2x04_P2.54mm_Vertical, B.Cu at (55.6, 105.7)
- moved J1 2.05 mm to (59.4, 65.0)
- moved J3 2.00 mm to (54.8, 81.0)
- moved J4 2.00 mm to (64.0, 81.0)
- moved J5 2.00 mm to (54.8, 96.0)
- moved J6 2.00 mm to (64.0, 96.0)
Connections:
- J1 pad 5: unconnected-(J1-Pad5) -> /A5
- J1 pad 6: unconnected-(J1-Pad6) -> /A6
- J1 pad 7: unconnected-(J1-Pad7) -> /A7
- J1 pad 8: unconnected-(J1-Pad8) -> /A8
- J2 pad 5: unconnected-(J2-Pad5) -> /B5
- J2 pad 6: unconnected-(J2-Pad6) -> /B6
- J2 pad 7: unconnected-(J2-Pad7) -> /B7
- J2 pad 8: unconnected-(J2-Pad8) -> /B8
Routing:
- net /B3: track 31.9 -> 48.0 mm
- net /A5: track 0.00 -> 11.8 mm
- net /B5: track 0.00 -> 11.8 mm
- net /A3: track 31.9 -> 43.2 mm
- net /A1: track 17.1 -> 26.8 mm
- net /B1: track 16.8 -> 26.0 mm
- net /B4: track 36.8 -> 45.6 mm
- net /A4: track 36.5 -> 44.5 mm
- net /B7: track 0.00 -> 6.69 mm
- net /A7: track 0.00 -> 6.69 mm
- net /A2: track 23.4 -> 30.1 mm
- net /B2: track 23.4 -> 30.0 mm
- net /B6: track 0.00 -> 4.67 mm
- net /A6: track 0.00 -> 4.67 mm
- net /B8: track 0.00 -> 3.62 mm
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Other:
- board text added: "1"
- board text added: "4"
- board text added: "5"
- board text added: "8"
- board text added: "QBreakout v1.0"
- board text removed: "J4"
- board text removed: "Quadraphone Breakout v1"
