File: Quadraphone_Controls_v3.kicad_sch (KiCad schematic)
At the start: 32 parts, among them J1 Conn_01x10_Female, J10 Pitch_In, J11 Mix_Out, J13 Conn_01x04_Male, J14 Conn_01x01_Male, J2 Conn_01x10_Female, J3 Conn_01x10_Female, J4 Conn_01x10_Female, J5 PWM_CV, J6 LFO_IN, J7 PWM_CV_In, J8 Synch_Signal_In, J9 Freq_Mod_In, SW1 Synch_Type, SW2 Output_Type, SW3 Output_Type

Commit message: Updates to controls Synch input protection
Parts:
- removed D2: 3d_Model_Panel, Custom_Footprints:3D_Dummy, symbol Mountjoy:3d_Model_Dummy
- removed R4: 10k, Resistor_SMD:R_0805_2012Metric, symbol Device:R_Small
- added R10, R8: 12k, Resistor_SMD:R_0805_2012Metric, symbol Device:R_Small
- added R3, R7, R9: 10k, Resistor_SMD:R_0805_2012Metric, symbol Device:R_Small
- added TP1: 2V_Test, Custom_Footprints:1mm_Test_Point, symbol Connector:TestPoint
- R4: renamed from R3; value 10k -> 12k
- R6: value 10k -> 12k
Connections:
- net 2V: now also TP1.1
- net GND: now also R10.2, R8.2; no longer R5.2
- net SYNCH_SIGNAL1: now also R3.1; no longer D3.2 (A), R4.1
- net SYNCH_SIGNAL2: now also R5.1; no longer D4.2 (A)
- net SYNCH_SIGNAL3: now also R7.1; no longer D5.2 (A), R5.1
- net SYNCH_SIGNAL4: now also R9.1; no longer D6.2 (A), R6.1
- net Synch1: now also R4.1
- net Synch2: now also R6.1
- net Synch3: now also R8.1
- net Synch4: now also R10.1
- new net: D3.2 (A), R3.2
- new net: D5.2 (A), R7.2
- new net: D6.2 (A), R9.2
- new net: D4.2 (A), R5.2
Other:
- moved on the sheet: D3, D4, D5, D6, R4

Commit message: Updated resistor values in VCO tuning circuits
Parts:
- removed D1: 3d_Model_Components, Custom_Footprints:3D_Dummy, symbol Mountjoy:3d_Model_Dummy
- added TP2: OctTest, Custom_Footprints:1mm_Test_Point, symbol Connector:TestPoint
- J1, J2, J3, J4: symbol Connector:Conn_01x10_Female -> Connector:Conn_01x10_Socket
- J13: symbol Connector:Conn_01x04_Male -> Connector:Conn_01x04_Pin
- J14: symbol Connector:Conn_01x01_Male -> Connector:Conn_01x01_Pin
- renumbered Fine_Tune2 to OctaveTrim1
Connections:
- net OCT_TUNE: now also TP2.1
Other:
- moved on the sheet: J1, J2, J3, J4, J7, J9
